File: projects/CAT_MEP/CAT_MEP.kicad_sch (KiCad schematic)
At the start: 12 parts, among them U1 TPS63051

Commit message: add Cat MEP und  alle outputjobs
Parts:
- added C11, C13, C14, C15, C16, C17: 100n, passive:C_0402, symbol db:capacitor/05.040.385.0
- added C12: 2u2, passive:C_0402, symbol db:capacitor/15.040.449.0
- added D1: PMEG2005CT, package:SOT-23, symbol db:diode/06.010.001
- added J1: USB_C_Receptacle_Molex_216990-0001, connector:USB_C_Receptacle_MidMnt_Molex_16_Contact_216990-0001, symbol db:connector/12.010.001
- added J2, J3: ConM-1x20, connector:PinHeader_1x20_P2.54mm_Vertical, symbol db:connector/12.020.020.0
- added J4: TC2030-IDC-NL, connector:TC2030-IDC-NL, symbol db:connector/12.011.001
- added R1, R2: 27R, passive:R_0402, symbol db:resistor/21.040.358.0
- added R3, R4: 5k1, passive:R_0402, symbol db:resistor/21.040.467.0
- added R5: 10k, passive:R_0402, symbol db:resistor/21.040.481.0
- added R6: 1k, passive:R_0402, symbol db:resistor/21.040.433.0
- added R7, R8: 3k3, passive:R_0402, symbol db:resistor/21.040.458.0
- added SW1: PTS815-SJM, switch:PTS815-Series, symbol db:switch/23.005.001
- added U2: RP2040, package:QFN-56-1EP_7x7mm_P0.4mm_EP3.2x3.2mm, symbol ic:RP2040
- added U3: W25Q16JV, package:USON_2x3x0.6mm, symbol db:ic/26.030.001
- added U4: SHT40-AD1B, package:SHT4x, symbol db:ic/26.040.010
- added Y1: CSTNE12M0GH5L000R0, discrete:Resonator_SMD_Murata_CSTxExxV-3Pin_3.0x1.1mm, symbol db:crystal/27.010.001
- U1: footprint ic:TPS63051 -> package:VQFN-12-1EP_2.5x2.5mm_P0.5mm; FP TPS63051 -> VQFN-12-1EP_2.5x2.5mm_P0.5mm; Modified 2024-02-14 10:59:50 -> 2024-02-15 09:53:02; Version 7 -> 10
- renumbered C7 to C1, C6 to C10, C9 to C2, C10 to C3, C8 to C4, C1 to C5, C2 to C6, C3 to C7, C4 to C8, C5 to C9
Connections:
- net GND: now also C2.2, C3.2, U1.10 (ILIM0), C11.2, C12.2, C13.2, C14.2, C15.2, C16.2, C17.2, J1.A1 (GND), J2.19, J2.20, J3.18, J3.19, J3.20, J4.5, R3.2, R4.2, SW1.1, U2.19 (TESTEN), U2.57 (VSS), U3.4 (GND), U4.4 (VSS), Y1.2
- net +3V3: now reaches C8.1
- net +3V3: now also C10.1, C2.1, C3.1, C5.1, C6.1, C7.1, C9.1, U1.4 (VOUT), U1.5 (FB), C11.1, C16.1, C17.1, J3.1, J3.2, J3.3, J4.1, R5.1, R7.1, R8.1, U2.1 (VDD), U2.10 (VDD), U2.22 (VDD), U2.33 (VDD), U2.42 (VDD), U2.43 (AVDD), U2.44 (VREG_VIN), U2.48 (USB_VDD), U2.49 (VDD), U3.8 (VCC), U4.3 (VDD)
- net Vin renamed VDD
- net VDD: now also D1.3 (K), D1.3 (K)
- new net: R6.2, SW1.2
- new net: J1.A5 (CC1), R4.1
- new net: J1.A6 (D+), J1.B6 (D+), R2.1
- new net: J1.A7 (D-), J1.B7 (D-), R1.1
- new net: J1.B5 (CC2), R3.1
- new net: U2.20 (XIN), Y1.1
- new net: U2.21 (XOUT), Y1.3
- new net: C12.1, C13.1, C14.1, U2.23 (DVVD), U2.45 (VREG_VOUT), U2.50 (DVVD)
- new net: U2.51 (SPI_SD3), U3.7 (~{R-H}_(IO3))
- new net: U2.53 (SPI_SD0), U3.5 (DI_(IO0))
- new net: U2.54 (SPI_SD2), U3.3 (~{WP}_(IO2))
- new net: U2.55 (SPI_SD1), U3.2 (D0(IO1))
- new net +5V: D1.1 (K), J2.1, J2.2
- new net A0: J2.3, U2.2 (GPIO0)
- new net A1: J2.4, U2.3 (GPIO1)
- new net A10: J2.13, U2.13 (GPIO10)
- new net A11: J2.14, U2.14 (GPIO11)
- new net A12: J2.15, R8.2, U2.15 (GPIO12), U4.1 (SDA)
- new net A13: J2.16, R7.2, U2.16 (GPIO13), U4.2 (SCL)
- new net A14: J2.17, U2.17 (GPIO14)
- new net A15: J2.18, U2.18 (GPIO15)
- new net A2: J2.5, U2.4 (GPIO2)
- new net A3: J2.6, U2.5 (GPIO3)
- new net A4: J2.7, U2.6 (GPIO4)
- new net A5: J2.8, U2.7 (GPIO5)
- new net A6: J2.9, U2.8 (GPIO6)
- new net A7: J2.10, U2.9 (GPIO7)
- new net A8: J2.11, U2.11 (GPIO8)
- new net A9: J2.12, U2.12 (GPIO9)
- new net B0: J3.4, U2.27 (GPIO16)
- new net B1: J3.5, U2.28 (GPIO17)
- new net B10: J3.14, U2.38 (GPIO26/ADC0)
- new net B11: J3.15, U2.39 (GPIO27/ADC1)
- new net B12: J3.16, U2.40 (GPIO28/ADC2)
- new net B13: J3.17, U2.41 (GPIO29/ADC3)
- new net B2: J3.6, U2.29 (GPIO18)
- new net B3: J3.7, U2.30 (GPIO19)
- new net B4: J3.8, U2.31 (GPIO20)
- new net B5: J3.9, U2.32 (GPIO21)
- new net B6: J3.10, U2.34 (GPIO22)
- new net B7: J3.11, U2.35 (GPIO23)
- new net B8: J3.12, U2.36 (GPIO24)
- new net B9: J3.13, U2.37 (GPIO25)
- new net CLK: U2.52 (SPI_SCLK), U3.6 (CLK)
- new net CS: R6.1, U2.56 (SPI_SS_N), U3.1 (~{CS})
- new net DM: R1.2, U2.46 (USB_DM)
- new net DP: R2.2, U2.47 (USB_DP)
- new net RESET: C15.1, J4.3, R5.2, U2.26 (RUN)
- new net SWD_CLK: J1.B8 (SBU2), J4.4, U2.24 (SWCLK)
- new net SWD_DIO: J1.A8 (SBU1), J4.2, U2.25 (SWDIO)
- new net VBUS: D1.2 (K), J1.A4 (VBUS)
- no-connect marks 0 -> 3
Other:
- moved on the sheet: C1, C10, C2, C3, C4, C5, C6, C7, C8, C9, U1
